File: PCB/Hexapod.kicad_pcb (KiCad board)
At the start: 4 copper layers, 100 x 100 mm, 11 parts, among them J1 Servo Driver In, J10 Out+, J2 Servo Driver Out, J3 Raspberry, J4 Servo Driver Out, J5 Servo Driver In, J6 Conn_02x06_Odd_Even, J7 IN-, J8 IN+, J9 Out-

Commit message: Update schematic and PCB
Parts:
- J6: value Conn_02x06_Odd_Even -> Pins
Connections:
- J1 pad 5: /OE -> unconnected-(J1-Pin_5-Pad5)
- J2 pad 2: /5V -> Net-(J2-Pin_2)
- J2 pad 3: /SCL -> Net-(J2-Pin_3)
- J2 pad 4: /SDA -> Net-(J2-Pin_4)
- J2 pad 5: /OE -> unconnected-(J2-Pin_5-Pad5)
- J4 pad 1: +BATT -> unconnected-(J4-Pin_1-Pad1)
- J4 pad 2: /5V -> unconnected-(J4-Pin_2-Pad2)
- J4 pad 3: /SCL -> unconnected-(J4-Pin_3-Pad3)
- J4 pad 4: /SDA -> unconnected-(J4-Pin_4-Pad4)
- J4 pad 5: /OE -> unconnected-(J4-Pin_5-Pad5)
- J4 pad 6: -BATT -> unconnected-(J4-Pin_6-Pad6)
- J5 pad 2: /5V -> Net-(J2-Pin_2)
- J5 pad 3: /SCL -> Net-(J2-Pin_3)
- J5 pad 4: /SDA -> Net-(J2-Pin_4)
- J5 pad 5: /OE -> unconnected-(J5-Pin_5-Pad5)
Routing:
- net Net-(J2-Pin_2): track 0.00 -> 72.1 mm
- net /5V: track 177.2 -> 105.1 mm
- net Net-(J2-Pin_4): track 0.00 -> 68.9 mm
- net /SCL: track 128.8 -> 61.2 mm
- net Net-(J2-Pin_3): track 0.00 -> 67.6 mm
- net /SDA: track 120.4 -> 57.2 mm
- net /OE: track 58.8 -> 0.00 mm
- net -BATT: track 145.2 -> 91.2 mm
